File: Apricot-Hard-Disk-Interface.kicad_sch (KiCad schematic)
At the start: 23 parts, among them J1 Motherboard Connector, J2 Expansion, J3 SD_CARD_READER, P1 Pico, U1 GAL16V8, U2 74AHCT244, U3 74LS245, U4 GAL16V8, U5 74LS245, U6 74LS373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

Commit message: Updated the PCB to the latest schematic and routed the PCB. Added Readme.md files
Parts:
- U3: value 74LS245 -> 74AHCT245
Changed lines of the file:
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@@
       (effects (font (size 1.27 1.27)) (justify right))
     )
-    (property "Value" "74LS245" (id 1) (at 108.585 162.814 90)
+    (property "Value" "74AHCT245" (id 1) (at 108.585 162.814 90)
       (effects (font (size 1.27 1.27)) (justify right))
     )
@@
     )
     (path "/1f67cb67-118d-4f11-96a3-bc4028b3a359"
-      (reference "U3") (unit 1) (value "74LS245") (footprint "Package_DIP:DIP-20_W7.62mm_Socket")
+      (reference "U3") (unit 1) (value "74AHCT245") (footprint "Package_DIP:DIP-20_W7.62mm_Socket")
     )
     (path "/a79178a7-e116-45e7-84d2-30a30f8bb515"
